Commit message: created V2 dual arm

File: dual_arm_configure/config/dual_arm.ros2_control.xacro (robot description, xacro)
@@ -19,5 +19,5 @@
         <state_interface name="velocity"/>
         <param name="can_id">0x01</param>
-        <param name="position_offset">-1374770</param>
+        <param name="position_offset">0</param>
       </joint>
       <joint name="joint2_right">
@@ -27,5 +27,5 @@
         <state_interface name="velocity"/>
         <param name="can_id">0x02</param>
-        <param name="position_offset">10668</param>
+        <param name="position_offset">0</param>
       </joint>
       <joint name="joint3_right">
@@ -35,5 +35,5 @@
         <state_interface name="velocity"/>
         <param name="can_id">0x03</param>
-        <param name="position_offset">565960</param>
+        <param name="position_offset">0</param>
       </joint>
       <joint name="joint4_right">
@@ -43,5 +43,5 @@
         <state_interface name="velocity"/>
         <param name="can_id">0x04</param>
-        <param name="position_offset">-610192</param>
+        <param name="position_offset">0</param>
       </joint>
       <joint name="joint5_right">
@@ -51,5 +51,5 @@
         <state_interface name="velocity"/>
         <param name="can_id">0x05</param>
-        <param name="position_offset">1319010</param>
+        <param name="position_offset">0</param>
       </joint>
       <joint name="joint6_right">
@@ -60,5 +60,4 @@
         <param name="can_id">0x06</param>
         <param name="position_offset">0</param>
-        <!-- <param name="position_offset">-1256290</param> -->
       </joint>
       <joint name="joint7_right">
@@ -69,5 +68,4 @@
         <param name="can_id">0x07</param>
         <param name="position_offset">0</param>
-        <!-- <param name="position_offset">-64386</param> -->
       </joint>
     </ros2_control>
@@ -89,5 +87,5 @@
           <state_interface name="velocity"/>
           <param name="can_id">0x01</param>
-          <param name="position_offset">-1441450</param>
+          <param name="position_offset">0</param>
         </joint>
         <joint name="joint2_left">
@@ -97,5 +95,5 @@
           <state_interface name="velocity"/>
           <param name="can_id">0x02</param>
-          <param name="position_offset">-1726200</param>
+          <param name="position_offset">0</param>
         </joint>
         <joint name="joint3_left">
@@ -105,5 +103,5 @@
           <state_interface name="velocity"/>
           <param name="can_id">0x03</param>
-          <param name="position_offset">-1708000</param>
+          <param name="position_offset">0</param>
         </joint>
         <joint name="joint4_left">
@@ -113,5 +111,5 @@
           <state_interface name="velocity"/>
           <param name="can_id">0x04</param>
-          <param name="position_offset">453945</param>
+          <param name="position_offset">0</param>
         </joint>
         <joint name="joint5_left">
@@ -121,5 +119,5 @@
           <state_interface name="velocity"/>
           <param name="can_id">0x05</param>
-          <param name="position_offset">-1427110</param>
+          <param name="position_offset">0</param>
         </joint>
         <joint name="joint6_left">
@@ -129,5 +127,5 @@
           <state_interface name="velocity"/>
           <param name="can_id">0x06</param>
-          <param name="position_offset">-177993</param>
+          <param name="position_offset">0</param>
         </joint>
         <joint name="joint7_left">
@@ -138,5 +136,4 @@
           <param name="can_id">0x07</param>
           <param name="position_offset">0</param>
-          <!-- <param name="position_offset">-475092</param> -->
         </joint>
     </ros2_control>

File: dual_arm_configure/config/dual_arm_demo.urdf.xacro (robot description, xacro)
@@ -8,6 +8,6 @@
   </xacro:dual_arm>
   <xacro:dual_arm_ros2_control
-    sim_left="true" can_interface_left="can0"
-    sim_right="true" can_interface_right="can1"
+    sim_left="false" can_interface_left="can0"
+    sim_right="false" can_interface_right="can1"
     namespace="upper_orin" />
 </robot>

File: dual_arm_description/urdf/dual_arm.urdf.xacro (robot description, xacro)
@@ -4,13 +4,16 @@
     <link name="arm_base_link">
       <inertial>
-        <origin xyz="-0.0049955 1.1496E-05 -0.010911" rpy="0 0 0" />
-        <mass value="1.8543" />
-        <inertia
-          ixx="0.015561"
-          ixy="-1.1941E-05"
-          ixz="-0.00041199"
-          iyy="0.011465"
-          iyz="-7.8472E-06"
-          izz="0.0059878" />
+        <origin
+          xyz="0.00422660431318732 0.0234645266440117 0.245520280917725"
+          rpy="0 0 0" />
+        <mass
+          value="5.9817893495402" />
+        <inertia
+          ixx="0.0763323573675301"
+          ixy="-1.0074625706827E-05"
+          ixz="0.00159918574737791"
+          iyy="0.0636485948623856"
+          iyz="2.44985620056427E-05"
+          izz="0.0205452676830648" />
       </inertial>
       <visual>
@@ -26,5 +29,5 @@
         <origin xyz="0 0 0" rpy="0 0 0" />
         <geometry>
-          <mesh filename="package://dual_arm_description/meshes/collision/base_link_simplify.STL" />
+          <mesh filename="package://dual_arm_description/meshes/collision/base_link.STL" />
         </geometry>
       </collision>
@@ -38,13 +41,16 @@
     <link name="link1_right">
       <inertial>
-        <origin xyz="0.00050131 1.9101E-07 -0.052638" rpy="0 0 0" />
-        <mass value="0.15855" />
-        <inertia
-          ixx="0.00021207"
-          ixy="-2.9917E-07"
-          ixz="3.54E-06"
-          iyy="0.00032023"
-          iyz="-2.3961E-07"
-          izz="0.00024019" />
+        <origin
+          xyz="-2.63462902565514E-05 0.0078456858397038 -0.0150193737682288"
+          rpy="0 0 0" />
+        <mass
+          value="1.80177628827918" />
+        <inertia
+          ixx="0.00125384727993194"
+          ixy="-1.9831651733611E-06"
+          ixz="-5.2634557942785E-07"
+          iyy="0.0012637095931909"
+          iyz="-2.91199249955174E-05"
+          izz="0.00129616591017272" />
       </inertial>
       <visual>
@@ -65,9 +71,8 @@
     </link>
     <joint name="joint1_right" type="revolute">
-      <!-- <origin xyz="0.0003839 0.124 0.012675" rpy="1.57079632679 3.14159265359 -0.003096" /> -->
-      <origin xyz="0.0003839 0.124 0.012675" rpy="1.57079632679 3.14159265359 0" />
+      <origin xyz="-0.0078 -0.155 0.32721" rpy="1.57079632679494 -1.57079632679494 0" />
       <parent link="arm_base_link" />
       <child link="link1_right" />
-      <axis xyz="0 0 -1" />
+      <axis xyz="0 0 1" />
       <limit
         lower="-3.14159265359"
@@ -78,13 +83,16 @@
     <link name="link2_right">
       <inertial>
-        <origin xyz="-0.029922 0.0026714 0.0026363" rpy="0 0 0" />
-        <mass value="0.33873" />
-        <inertia
-          ixx="0.00073505"
-          ixy="1.7822E-06"
-          ixz="-2.2248E-05"
-          iyy="0.00068697"
-          iyz="3.5427E-06"
-          izz="0.00044803" />
+        <origin
+          xyz="-0.0184912045878147 0.00162452489349674 0.013616878292953"
+          rpy="0 0 0" />
+        <mass
+          value="0.722746235912474" />
+        <inertia
+          ixx="0.00108593997275333"
+          ixy="1.84897338808204E-06"
+          ixz="-3.09028194254925E-05"
+          iyy="0.00101515721108136"
+          iyz="4.99580004142565E-06"
+          izz="0.000753458785916066" />
       </inertial>
       <visual>
@@ -105,8 +113,8 @@
     </link>
     <joint name="joint2_right" type="revolute">
-      <origin xyz="0 0 -0.056" rpy="3.14159265359 -1.57079632679 0" />
+      <origin xyz="0 0 0.054" rpy="0 1.5707963267949 0" />
       <parent link="link1_right" />
       <child link="link2_right" />
-      <axis xyz="0 0 1" />
+      <axis xyz="0 0 -1" />
       <limit
         lower="-1.57079632679"
@@ -117,13 +125,16 @@
     <link name="link3_right">
       <inertial>
-        <origin xyz="-0.0058267 -0.0016701 0.11259" rpy="0 0 0" />
-        <mass value="0.34337" />
-        <inertia
-          ixx="0.0016463"
-          ixy="-1.8501E-05"
-          ixz="0.00013984"
-          iyy="0.0016097"
-          iyz="4.8636E-05"
-          izz="0.00049751" />
+        <origin
+          xyz="0.00248327358203637 0.000983930202917094 0.0848422618072029"
+          rpy="0 0 0" />
+        <mass
+          value="1.73968703689437" />
+        <inertia
+          ixx="0.00293287578739714"
+          ixy="-4.78768415153896E-05"
+          ixz="-0.000146666097337501"
+          iyy="0.00269293929456573"
+          iyz="-6.8741663865335E-05"
+          izz="0.00158103557348051" />
       </inertial>
       <visual>
@@ -144,5 +155,5 @@
     </link>
     <joint name="joint3_right" type="revolute">
-      <origin xyz="-0.0705 0 0" rpy="1.57079632679 3.14159265359 -1.57079632679" />
+      <origin xyz="-0.07 0 0" rpy="0 -1.57067311902631 0" />
       <parent link="link2_right" />
       <child link="link3_right" />
@@ -156,13 +167,16 @@
     <link name="link4_right">
       <inertial>
-        <origin xyz="6.1575E-07 -0.011496 -0.0028054" rpy="0 0 0" />
-        <mass value="0.13904" />
-        <inertia
-          ixx="0.00024464"
-          ixy="1.3836E-07"
-          ixz="4.0416E-08"
-          iyy="0.00015494"
-          iyz="-1.3471E-06"
-          izz="0.00017092" />
+        <origin
+          xyz="-7.95973702305552E-05 -0.0209082375496418 -0.00839273362275947"
+          rpy="0 0 0" />
+        <mass
+          value="1.29895950213977" />
+        <inertia
+          ixx="0.00236791349815647"
+          ixy="1.40731293258229E-06"
+          ixz="3.26442183375437E-06"
+          iyy="0.000772031871168032"
+          iyz="-1.41965703385309E-05"
+          izz="0.00230845350224412" />
       </inertial>
       <visual>
@@ -183,5 +197,5 @@
     </link>
     <joint name="joint4_right" type="revolute">
-      <origin xyz="-0.038197 0 0.19969" rpy="-1.57079632679 0 3.14159265359" />
+      <origin xyz="-0.03857 0 0.23768" rpy="0 1.5707963267949 -1.5707963267949" />
       <parent link="link3_right" />
       <child link="link4_right" />
@@ -189,5 +203,5 @@
       <limit
         lower="-2.44"
-        upper="1.0"
+        upper="0.698131701"
         effort="0"
         velocity="0.436332313" />
@@ -195,13 +209,16 @@
     <link name="link5_right">
       <inertial>
-        <origin xyz="1.9806E-06 0.0018081 -0.078642" rpy="0 0 0" />
-        <mass value="0.14999" />
-        <inertia
-          ixx="0.00038781"
-          ixy="5.3153E-09"
-          ixz="-3.7041E-09"
-          iyy="0.00035795"
-          iyz="1.2827E-05"
-          izz="0.00015133" />
+        <origin
+          xyz="6.30477802943119E-05 0.00086654932953717 -0.0916349080676876"
+          rpy="0 0 0" />
+        <mass
+          value="0.943914536026674" />
+        <inertia
+          ixx="0.000931990246154717"
+          ixy="-9.21631995424494E-06"
+          ixz="-2.51581497978434E-06"
+          iyy="0.000811077416357626"
+          iyz="-3.8715241803587E-05"
+          izz="0.000572990604772896" />
       </inertial>
       <visual>
@@ -222,5 +239,5 @@
     </link>
     <joint name="joint5_right" type="revolute">
-      <origin xyz="0 -0.067 0" rpy="-1.57079632679 0 0" />
+      <origin xyz="-0.175 0 0" rpy="0 -1.5707963267949 0" />
       <parent link="link4_right" />
       <child link="link5_right" />
@@ -234,13 +251,16 @@
     <link name="link6_right">
       <inertial>
-        <origin xyz="-0.023745 -0.0018091 0.0026342" rpy="0 0 0" />
-        <mass value="0.14924" />
-        <inertia
-          ixx="0.00015555"
-          ixy="-9.0013E-06"
-          ixz="-3.6227E-06"
-          iyy="0.00021426"
-          iyz="-7.7162E-07"
-          izz="0.00022953" />
+        <origin
+          xyz="0.00799400089214897 -0.00109797731745931 0.00802800673798493"
+          rpy="0 0 0" />
+        <mass
+          value="0.87461121686283" />
+        <inertia
+          ixx="0.000482453783893589"
+          ixy="2.78696828473613E-05"
+          ixz="-1.16479121693327E-05"
+          iyy="0.000519252452409952"
+          iyz="2.15614721648117E-07"
+          izz="0.000655950625877922" />
       </inertial>
       <visual>
@@ -261,5 +281,5 @@
     </link>
     <joint name="joint6_right" type="revolute">
-      <origin xyz="0 0 -0.133" rpy="1.57079632679 -1.57079632679 0" />
+      <origin xyz="0 0 0.135" rpy="0 -1.5707963267949 0" />
       <parent link="link5_right" />
       <child link="link6_right" />
@@ -273,13 +293,16 @@
     <link name="link7_right">
       <inertial>
-        <origin xyz="8.607E-07 0.0034748 -0.0017068" rpy="0 0 0" />
-        <mass value="0.082918" />
-        <inertia
-          ixx="5.7371E-05"
-          ixy="-3.2078E-09"
-          ixz="-5.1253E-10"
-          iyy="5.6287E-05"
-          iyz="-5.9283E-07"
-          izz="6.5419E-05" />
+        <origin
+          xyz="0.00118014491083041 -0.000343927719202997 0.00924911342229717"
+          rpy="0 0 0" />
+        <mass
+          value="0.755429789120553" />
+        <inertia
+          ixx="0.000269322287342564"
+          ixy="6.31271638827115E-06"
+          ixz="-7.63621824391722E-08"
+          iyy="0.000289179185961173"
+          iyz="1.47888072820137E-08"
+          izz="0.000297353940351334" />
       </inertial>
       <visual>
@@ -300,8 +323,8 @@
     </link>
     <joint name="joint7_right" type="revolute">
-      <origin xyz="-0.065 -0.0015 0" rpy="1.57079632679 1.57079632679 3.14159265359" />
+      <origin xyz="0.067 0 0" rpy="-1.5707963267949 0 0" />
       <parent link="link6_right" />
       <child link="link7_right" />
-      <axis xyz="0 0 -1" />
+      <axis xyz="0 0 1" />
       <limit
         lower="-1.05"
@@ -312,13 +335,16 @@
     <link name="link1_left">
       <inertial>
-        <origin xyz="0.00050131 1.9101E-07 -0.052638" rpy="0 0 0" />
-        <mass value="0.15855" />
-        <inertia
-          ixx="0.00021207"
-          ixy="-2.9917E-07"
-          ixz="3.54E-06"
-          iyy="0.00032023"
-          iyz="-2.3961E-07"
-          izz="0.00024019" />
+        <origin
+          xyz="-1.38487613492444E-05 -0.00220692224137892 0.00921894631138384"
+          rpy="0 0 0" />
+        <mass
+          value="0.519339306262197" />
+        <inertia
+          ixx="0.000497409399128485"
+          ixy="1.04568338202191E-06"
+          ixz="6.91360153863362E-08"
+          iyy="0.000419809278764117"
+          iyz="-1.06406718218775E-05"
+          izz="0.000437145559325128" />
       </inertial>
       <visual>
@@ -339,5 +365,5 @@
     </link>
     <joint name="joint1_left" type="revolute">
-      <origin xyz="-0.0003839 -0.124 0.012675" rpy="1.57079632679 3.14159265359 3.14159265359" />
+      <origin xyz="-0.0078 0.155 0.32721" rpy="0 -1.57079632679494 -1.57079632679494" />
       <parent link="arm_base_link" />
       <child link="link1_left" />
@@ -351,13 +377,16 @@
     <link name="link2_left">
       <inertial>
-        <origin xyz="-0.029922 -0.0026714 -0.0026363" rpy="0 0 0" />
-        <mass value="0.33873" />
-        <inertia
-          ixx="0.00073505"
-          ixy="-1.7822E-06"
-          ixz="2.2248E-05"
-          iyy="0.00068697"
-          iyz="3.5427E-06"
-          izz="0.00044803" />
+        <origin
+          xyz="0.005428504454426 0.0228357969273356 0.00572697696991797"
+          rpy="0 0 0" />
+        <mass
+          value="0.254319595126366" />
+        <inertia
+          ixx="0.000415729754126609"
+          ixy="1.31927673128639E-06"
+          ixz="3.33686056832701E-06"
+          iyy="0.000437161837114042"
+          iyz="1.09061160250672E-05"
+          izz="0.00033601383844043" />
       </inertial>
       <visual>
@@ -378,8 +407,8 @@
     </link>
     <joint name="joint2_left" type="revolute">
-      <origin xyz="0 0 -0.056" rpy="0 -1.57079632679 0" />
+      <origin xyz="0 0 0.054" rpy="0 1.5707963267949 0" />
       <parent link="link1_left" />
       <child link="link2_left" />
-      <axis xyz="0 0 -1" />
+      <axis xyz="0 0 1" />
       <limit
         lower="-1.57079632679"
@@ -390,13 +419,16 @@
     <link name="link3_left">
       <inertial>
-        <origin xyz="-0.0058267 -0.0016701 0.11259" rpy="0 0 0" />
-        <mass value="0.34337" />
-        <inertia
-          ixx="0.0016463"
-          ixy="-1.8501E-05"
-          ixz="0.00013984"
-          iyy="0.0016097"
-          iyz="4.8636E-05"
-          izz="0.00049751" />
+        <origin
+          xyz="0.00322397114526773 0.000846637475657469 0.0985307535142525"
+          rpy="0 0 0" />
+        <mass
+          value="0.676008865226733" />
+        <inertia
+          ixx="0.00175191112419296"
+          ixy="-1.70722602314306E-05"
+          ixz="-0.000113910532811989"
+          iyy="0.00172370166259428"
+          iyz="-2.23111533397412E-05"
+          izz="0.000671070067083804" />
       </inertial>
       <visual>
@@ -417,5 +449,5 @@
     </link>
     <joint name="joint3_left" type="revolute">
-      <origin xyz="-0.0705 0 0" rpy="1.57079632679 0 -1.57079632679" />
+      <origin xyz="-0.07 0 0" rpy="0 -1.5707963267949 0" />
       <parent link="link2_left" />
       <child link="link3_left" />
@@ -429,13 +461,16 @@
     <link name="link4_left">
       <inertial>
-        <origin xyz="-6.1575E-07 -0.011496 0.0028054" rpy="0 0 0" />
-        <mass value="0.13904" />
-        <inertia
-          ixx="0.00024464"
-          ixy="-1.3836E-07"
-          ixz="4.0416E-08"
-          iyy="0.00015494"
-          iyz="1.3471E-06"
-          izz="0.00017092" />
+        <origin
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